File: P-01_power_input/P-01-R_power_adapter.kicad_pcb (KiCad board)
At the start: 2 copper layers, 22 x 51 mm, 16 parts, among them J1 POWER_A, J2 POWER_B, J3 CHAIN_TOP, J4 +5V_OUT, J5 POWER_IN, J6 CHAIN_BOTTOM

Commit message: Fix P-01 file associations, diodes, erc check
Parts:
- D1, D2, D3: value 1N5819 -> 1N5819HW
